File: Keyboard.kicad_pcb (KiCad board)
At the start: 2 copper layers, 354.8 x 131 mm, 199 parts, among them SW1 SW_Push, SW10 SW_Push, SW11 SW_Push, SW12 SW_Push, SW13 SW_Push, SW14 SW_Push, SW15 SW_Push, SW16 SW_Push, SW17 SW_Push, SW18 SW_Push, SW19 SW_Push, SW2 SW_Push, SW20 SW_Push, SW21 SW_Push, SW22 SW_Push, SW23 SW_Push, SW24 SW_Push, SW25 SW_Push, SW26 SW_Push, SW27 SW_Push, SW28 SW_Push, SW29 SW_Push, SW3 SW_Push, SW30 SW_Push, SW31 SW_Push, SW32 SW_Push, SW33 SW_Push, SW34 SW_Push, SW35 SW_Push, SW36 SW_Push, SW37 SW_Push, SW38 SW_Push, SW39 SW_Push, SW4 SW_Push, SW40 SW_Push, SW41 SW_Push, SW42 SW_Push, SW43 SW_Push, SW44 SW_Push, SW45 SW_Push, SW46 SW_Push, SW47 SW_Push, SW48 SW_Push, SW49 SW_Push, SW5 SW_Push, SW50 SW_Push, SW51 SW_Push, SW52 SW_Push, SW53 SW_Push, SW54 SW_Push, SW55 SW_Push, SW56 SW_Push, SW57 SW_Push, SW58 SW_Push, SW59 SW_Push, SW6 SW_Push, SW60 SW_Push, SW61 SW_Push, SW62 SW_Push, SW63 SW_Push, SW64 SW_Push, SW65 SW_Push, SW66 SW_Push, SW67 SW_Push, SW68 SW_Push, SW69 SW_Push, SW7 SW_Push, SW70 SW_Push, SW71 SW_Push, SW72 SW_Push, SW73 SW_Push, SW74 SW_Push, SW75 SW_Push, SW76 SW_Push, SW77 SW_Push, SW78 SW_Push, SW79 SW_Push, SW8 SW_Push, SW80 SW_Push, SW81 SW_Push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

Commit message: added holes to my pcb
Routing:
- net Row 0: track 461.9 -> 464.5 mm
- net Row 5: track 368.5 -> 367.0 mm
Other:
- outline, holes or cut-outs redrawn
Changed lines of the file:
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@@
 		)
 	)
+	(gr_circle
+		(center 175.26 121.6)
+		(end 177.46 121.6)
+		(stroke
+			(width 0.05)
+			(type default)
+		)
+		(fill none)
+		(layer "Edge.Cuts")
+	)
+	(gr_circle
+		(center 318.19 64.28)
+		(end 320.39 64.28)
+		(stroke
+			(width 0.05)
+			(type default)
+		)
+		(fill none)
+		(layer "Edge.Cuts")
+	)
 	(gr_rect
 		(start -23.8125 14.2875)
@@
 		(layer "Edge.Cuts")
 	)
+	(gr_circle
+		(center 151.44 45.4)
+		(end 153.64 45.4)
+		(stroke
+			(width 0.05)
+			(type default)
+		)
+		(fill none)
+		(layer "Edge.Cuts")
+	)
+	(gr_circle
+		(center 237.17 83.5)
+		(end 239.37 83.5)
+		(stroke
+			(width 0.05)
+			(type default)
+		)
+		(fill none)
+		(layer "Edge.Cuts")
+	)
+	(gr_circle
+		(center 299.12 121.6)
+		(end 301.32 121.6)
+		(stroke
+			(width 0.05)
+			(type default)
+		)
+		(fill none)
+		(layer "Edge.Cuts")
+	)
+	(gr_circle
+		(center 227.64 45.4)
+		(end 229.84 45.4)
+		(stroke
+			(width 0.05)
+			(type default)
+		)
+		(fill none)
+		(layer "Edge.Cuts")
+	)
+	(gr_circle
+		(center 241.93 121.6)
+		(end 244.13 121.6)
+		(stroke
+			(width 0.05)
+			(type default)
+		)
+		(fill none)
+		(layer "Edge.Cuts")
+	)
+	(gr_circle
+		(center 280.02 45.25)
+		(end 282.22 45.25)
+		(stroke
+			(width 0.05)
+			(type default)
+		)
+		(fill none)
+		(layer "Edge.Cuts")
+	)
+	(gr_circle
+		(center -0.95 45.4)
+		(end 1.25 45.4)
+		(stroke
+			(width 0.05)
+			(type default)
+		)
+		(fill none)
+		(layer "Edge.Cuts")
+	)
+	(gr_circle
+		(center 75.25 45.41)
+		(end 77.45 45.41)
+		(stroke
+			(width 0.05)
+			(type default)
+		)
+		(fill none)
+		(layer "Edge.Cuts")
+	)
+	(gr_circle
+		(center 84.77 83.47)
+		(end 86.97 83.47)
+		(stroke
+			(width 0.05)
+			(type default)
+		)
+		(fill none)
+		(layer "Edge.Cuts")
+	)
+	(gr_circle
+		(center 8.57 83.5)
+		(end 10.77 83.5)
+		(stroke
+			(width 0.05)
+			(type default)
+		)
+		(fill none)
+		(layer "Edge.Cuts")
+	)
+	(gr_circle
+		(center 99.06 121.6)
+		(end 101.26 121.6)
+		(stroke
+			(width 0.05)
+			(type default)
+		)
+		(fill none)
+		(layer "Edge.Cuts")
+	)
+	(gr_circle
+		(center 160.97 83.5)
+		(end 163.17 83.5)
+		(stroke
+			(width 0.05)
+			(type default)
+		)
+		(fill none)
+		(layer "Edge.Cuts")
+	)
+	(gr_circle
+		(center 3.81 121.61)
+		(end 6.01 121.61)
+		(stroke
+			(width 0.05)
+			(type default)
+		)
+		(fill none)
+		(layer "Edge.Cuts")
+	)
 	(gr_text "@kaipereira gh"
 		(at 242.8875 22.621875 0)
@@
 	)
 	(segment
-		(start 231.995239 44.035239)
-		(end 280.245801 44.035239)
+		(start 293.936875 51.026875)
+		(end 293.936875 44.200625)
 		(width 0.2)
 		(layer "F.Cu")
@@
 	)
 	(segment
-		(start 293.936875 51.026875)
-		(end 293.936875 44.200625)
+		(start 290.5125 54.45125)
+		(end 293.936875 51.026875)
 		(width 0.2)
 		(layer "F.Cu")
@@
 	)
 	(segment
-		(start 290.5125 54.45125)
-		(end 293.936875 51.026875)
+		(start 230.23 42.27)
+		(end 282.01104 42.27)
 		(width 0.2)
 		(layer "F.Cu")
@@
 	)
 	(segment
+		(start 227.6475 39.6875)
+		(end 230.23 42.27)
+		(width 0.2)
+		(layer "F.Cu")
+		(net 1)
+	)
+	(segment
+		(start 283.799584 40.481456)
+		(end 285.75 40.481456)
+		(width 0.2)
+		(layer "F.Cu")
+		(net 1)
+	)
+	(segment
 		(start 302.786875 31.218649)
 		(end 302.786875 28.705)
@@
 	)
 	(segment
-		(start 283.799584 40.481456)
-		(end 285.75 40.481456)
-		(width 0.2)
-		(layer "F.Cu")
-		(net 1)
-	)
-	(segment
 		(start 288.331069 54.45125)
 		(end 290.5125 54.45125)
@@
 	)
 	(segment
-		(start 280.245801 44.035239)
+		(start 282.01104 42.27)
 		(end 283.799584 40.481456)
 		(width 0.2)
@@
 	)
 	(segment
-		(start 227.6475 39.6875)
-		(end 231.995239 44.035239)
-		(width 0.2)
-		(layer "F.Cu")
-		(net 1)
-	)
-	(segment
 		(start 302.786875 28.705)
 		(end 302.656875 28.575)
@@
 	)
 	(segment
-		(start 287.893125 80.724375)
-		(end 287.893125 69.294375)
+		(start 290.60625 66.58125)
+		(end 303.7825 66.58125)
 		(width 0.2)
 		(layer "F.Cu")
@@
 	)
 	(segment
-		(start 288.46 114.7875)
-		(end 288.46 81.29125)
+		(start 303.7825 66.58125)
+		(end 308.2925 62.07125)
 		(width 0.2)
 		(layer "F.Cu")
@@
 	)
 	(segment
-		(start 289.56 115.8875)
-		(end 288.46 114.7875)
+		(start 284.74 111.0675)
+		(end 284.74 83.8775)
 		(width 0.2)
 		(layer "F.Cu")
@@
 	)
 	(segment
-		(start 290.60625 66.58125)
-		(end 303.7825 66.58125)
+		(start 308.2925 62.07125)
+		(end 308.2925 61.120973)
 		(width 0.2)
 		(layer "F.Cu")
@@
 	)
 	(segment
-		(start 308.2925 62.07125)
-		(end 308.2925 61.120973)
+		(start 289.56 115.8875)
+		(end 284.74 111.0675)
 		(width 0.2)
 		(layer "F.Cu")
@@
 	)
 	(segment
-		(start 321.945 26.19375)
-		(end 324.248125 28.496875)
+		(start 287.893125 80.724375)
+		(end 287.893125 69.294375)
 		(width 0.2)
 		(layer "F.Cu")
@@
 	)
 	(segment
-		(start 324.248125 42.940625)
-		(end 321.945 45.24375)
+		(start 287.893125 69.294375)
+		(end 290.60625 66.58125)
 		(width 0.2)
 		(layer "F.Cu")
@@
 	)
 	(segment
-		(start 308.2925 61.120973)
-		(end 317.025973 52.3875)
+		(start 321.945 26.19375)
+		(end 324.248125 28.496875)
 		(width 0.2)
 		(layer "F.Cu")
@@
 	)
 	(segment
-		(start 287.893125 69.294375)
-		(end 290.60625 66.58125)
+		(start 284.74 83.8775)
+		(end 287.893125 80.724375)
 		(width 0.2)
 		(layer "F.Cu")
@@
 	)
 	(segment
-		(start 288.46 81.29125)
-		(end 287.893125 80.724375)
+		(start 324.248125 42.940625)
+		(end 321.945 45.24375)
 		(width 0.2)
 		(layer "F.Cu")
@@
 	)
 	(segment
-		(start 319.789274 52.3875)
-		(end 321.945 50.231774)
+		(start 308.2925 61.120973)
+		(end 317.025973 52.3875)
 		(width 0.2)
 		(layer "F.Cu")
@@
 	)
 	(segment
-		(start 317.025973 52.3875)
-		(end 319.789274 52.3875)
+		(start 319.789274 52.3875)
+		(end 321.945 50.231774)
 		(width 0.2)
 		(layer "F.Cu")
@@
 	)
 	(segment
-		(start 303.7825 66.58125)
-		(end 308.2925 62.07125)
+		(start 317.025973 52.3875)
+		(end 319.789274 52.3875)
 		(width 0.2)
 		(layer "F.Cu")
@@
 	)
 	(segment
-		(start 189.005 117.5675)
-		(end 188.11875 116.68125)
-		(width 0.2)
-		(layer "B.Cu")
-		(net 99)
-	)
-	(segment
 		(start 177.8 106.3625)
 		(end 178.59375 107.15625)
@@
 	)
 	(segment
-		(start 163.5125 19.4625)
-		(end 163.5125 30.95625)
-		(width 0.2)
-		(layer "B.Cu")
-		(net 99)
-	)
-	(segment
-		(start 188.11875 116.68125)
-		(end 188.11875 114.3)
+		(start 188.11875 114.3)
+		(end 187.325 113.50625)
 		(width 0.2)
 		(layer "B.Cu")
@@
 	)
 	(segment
-		(start 187.325 113.50625)
-		(end 187.325 106.9975)
+		(start 163.5125 19.4625)
+		(end 163.5125 30.95625)
 		(width 0.2)
 		(layer "B.Cu")
@@
 	)
 	(segment
-		(start 301.625 126.0475)
-		(end 293.145 117.5675)
+		(start 290.7375 117.5675)
+		(end 189.005 117.5675)
 		(width 0.2)
 		(layer "B.Cu")
@@
 	)
 	(segment
+		(start 189.005 117.5675)
+		(end 188.11875 116.68125)
+		(width 0.2)
+		(layer "B.Cu")
+		(net 99)
+	)
+	(segment
+		(start 301.625 126.0475)
+		(end 299.2175 126.0475)
+		(width 0.2)
+		(layer "B.Cu")
+		(net 99)
+	)
+	(segment
 		(start 164.30625 18.66875)
 		(end 163.5125 19.4625)
@@
 	)
 	(segment
+		(start 188.11875 116.68125)
+		(end 188.11875 114.3)
+		(width 0.2)
+		(layer "B.Cu")
+		(net 99)
+	)
+	(segment
 		(start 290.056865 40.31125)
 		(end 286.148125 36.40251)
@@
 	)
 	(segment
-		(start 163.5125 68.2625)
-		(end 164.30625 69.05625)
+		(start 187.325 113.50625)
+		(end 187.325 106.9975)
 		(width 0.2)
 		(layer "B.Cu")
@@
 	)
 	(segment
-		(start 284.55 18.66875)
-		(end 164.30625 18.66875)
+		(start 163.5125 68.2625)
+		(end 164.30625 69.05625)
 		(width 0.2)
 		(layer "B.Cu")
@@
 	)
 	(segment
-		(start 293.145 117.5675)
-		(end 189.005 117.5675)
+		(start 284.55 18.66875)
+		(end 164.30625 18.66875)
 		(width 0.2)
 		(layer "B.Cu")
@@
 	)
 	(segment
-		(start 188.11875 114.3)
-		(end 187.325 113.50625)
+		(start 286.148125 33.29625)
+		(end 284.55 31.698125)
 		(width 0.2)
 		(layer "B.Cu")
@@
 	)
 	(segment
-		(start 286.148125 33.29625)
-		(end 284.55 31.698125)
+		(start 299.2175 126.0475)
+		(end 290.7375 117.5675)
 		(width 0.2)
 		(layer "B.Cu")

Commit message: fix some drc errors
Routing:
- net Col 7: track 434.1 -> 432.9 mm
- net Col 6: track 445.2 -> 444.2 mm
Other:
- outline, holes or cut-outs redrawn
Changed lines of the file:
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@@
 	)
 	(gr_circle
-		(center 280.02 45.25)
-		(end 282.22 45.25)
+		(center 279.21 45.25)
+		(end 281.41 45.25)
 		(stroke
 			(width 0.05)
@@
 	)
 	(segment
-		(start 308.2925 16.35125)
-		(end 308.95625 15.6875)
-		(width 0.2)
-		(layer "B.Cu")
-		(net 90)
-	)
-	(segment
 		(start -3.175 68.8975)
 		(end -3.175 87.3125)
@@
 	)
 	(segment
-		(start -3.175 87.3125)
-		(end -2.38125 88.10625)
+		(start -5.3625 14.8875)
+		(end -7.9375 17.4625)
 		(width 0.2)
 		(layer "B.Cu")
@@
 	)
 	(segment
-		(start -7.9375 19.84375)
-		(end -7.9375 30.7975)
+		(start -3.175 87.3125)
+		(end -2.38125 88.10625)
 		(width 0.2)
 		(layer "B.Cu")
@@
 	)
 	(segment
-		(start -5.3625 14.8875)
-		(end -7.14375 16.66875)
-		(width 0.2)
-		(layer "B.Cu")
-		(net 90)
-	)
-	(segment
 		(start -0.79375 106.3625)
 		(end 0 107.15625)
@@
 	)
 	(segment
-		(start 308.95625 15.6875)
-		(end 308.95625 14.8875)
-		(width 0.2)
-		(layer "B.Cu")
-		(net 90)
-	)
-	(segment
-		(start 308.95625 14.8875)
-		(end -5.3625 14.8875)
-		(width 0.2)
-		(layer "B.Cu")
-		(net 90)
-	)
-	(segment
 		(start -6.985 68.8975)
 		(end -3.175 68.8975)
@@
 	)
 	(segment
+		(start -7.9375 17.4625)
+		(end -7.9375 30.7975)
+		(width 0.2)
+		(layer "B.Cu")
+		(net 90)
+	)
+	(segment
 		(start -4.7625 126.20625)
 		(end -4.92125 126.0475)
@@
 	)
 	(segment
+		(start 308.95625 15.6875)
+		(end 308.95625 14.8875)
+		(width 0.2)
+		(layer "B.Cu")
+		(net 90)
+	)
+	(segment
 		(start -2.38125 88.10625)
 		(end -2.2225 87.9475)
@@
 	)
 	(segment
-		(start -7.14375 19.05)
-		(end -7.9375 19.84375)
+		(start 308.95625 14.8875)
+		(end -5.3625 14.8875)
 		(width 0.2)
 		(layer "B.Cu")
@@
 	)
 	(segment
-		(start -7.14375 16.66875)
-		(end -7.14375 19.05)
+		(start 308.2925 16.35125)
+		(end 308.95625 15.6875)
 		(width 0.2)
 		(layer "B.Cu")
@@
 	)
 	(segment
-		(start 130.96875 119.0625)
-		(end 130.175 118.26875)
-		(width 0.2)
-		(layer "B.Cu")
-		(net 96)
-	)
-	(segment
 		(start 115.8875 68.8975)
 		(end 115.8875 87.3125)
@@
 	)
 	(segment
+		(start 130.96875 118.8)
+		(end 130.96875 119.0625)
+		(width 0.2)
+		(layer "B.Cu")
+		(net 96)
+	)
+	(segment
 		(start 123.825 107.15625)
 		(end 123.98375 106.9975)
@@
 	)
 	(segment
+		(start 130.175 118.26875)
+		(end 130.175 106.9975)
+		(width 0.2)
+		(layer "B.Cu")
+		(net 96)
+	)
+	(segment
+		(start 130.96875 119.0625)
+		(end 130.175 118.26875)
+		(width 0.2)
+		(layer "B.Cu")
+		(net 96)
+	)
+	(segment
 		(start 285.75 25.844385)
 		(end 285.75 17.46875)
@@
 	)
 	(segment
-		(start 107.15625 17.46875)
-		(end 106.3625 18.2625)
+		(start 203.488649 118.8)
+		(end 130.96875 118.8)
 		(width 0.2)
 		(layer "B.Cu")
@@
 	)
 	(segment
-		(start 232.56875 126.0475)
-		(end 210.736149 126.0475)
+		(start 107.15625 17.46875)
+		(end 106.3625 18.2625)
 		(width 0.2)
 		(layer "B.Cu")
@@
 	)
 	(segment
-		(start 130.96875 121.44375)
-		(end 130.96875 119.0625)
-		(width 0.2)
-		(layer "B.Cu")
-		(net 96)
-	)
-	(segment
 		(start 120.65 106.3625)
 		(end 121.44375 107.15625)
@@
 	)
 	(segment
-		(start 130.175 118.26875)
-		(end 130.175 106.9975)
-		(width 0.2)
-		(layer "B.Cu")
-		(net 96)
-	)
-	(segment
 		(start 290.056865 30.15125)
 		(end 285.75 25.844385)
@@
 	)
 	(segment
-		(start 210.736149 126.0475)
-		(end 206.132399 121.44375)
+		(start 232.56875 126.0475)
+		(end 210.736149 126.0475)
 		(width 0.2)
 		(layer "B.Cu")
@@
 	)
 	(segment
-		(start 206.132399 121.44375)
-		(end 130.96875 121.44375)
+		(start 116.68125 88.10625)
+		(end 119.0625 88.10625)
 		(width 0.2)
 		(layer "B.Cu")
@@
 	)
 	(segment
-		(start 116.68125 88.10625)
-		(end 119.0625 88.10625)
+		(start 210.736149 126.0475)
+		(end 203.488649 118.8)
 		(width 0.2)
 		(layer "B.Cu")
@@
 	)
 	(segment
+		(start 149.3925 118.3675)
+		(end 149.225 118.2)
+		(width 0.2)
+		(layer "B.Cu")
+		(net 97)
+	)
+	(segment
 		(start 308.2925 39.21125)
 		(end 305.722319 39.21125)
@@
 	)
 	(segment
-		(start 256.38125 126.0475)
-		(end 254.98125 124.6475)
+		(start 209.901835 124.6475)
+		(end 203.621835 118.3675)
 		(width 0.2)
 		(layer "B.Cu")
@@
 	)
 	(segment
-		(start 150.01875 121.04375)
-		(end 149.225 120.25)
+		(start 256.38125 126.0475)
+		(end 254.98125 124.6475)
 		(width 0.2)
 		(layer "B.Cu")
@@
 	)
 	(segment
+		(start 149.225 118.2)
+		(end 149.225 106.9975)
+		(width 0.2)
+		(layer "B.Cu")
+		(net 97)
+	)
+	(segment
 		(start 142.875 107.15625)
 		(end 143.03375 106.9975)
@@
 	)
 	(segment
-		(start 206.298085 121.04375)
-		(end 150.01875 121.04375)
-		(width 0.2)
-		(layer "B.Cu")
-		(net 97)
-	)
-	(segment
 		(start 128.74625 68.8975)
 		(end 134.9375 68.8975)
@@
 	)
 	(segment
-		(start 254.98125 124.6475)
-		(end 209.901835 124.6475)
-		(width 0.2)
-		(layer "B.Cu")
-		(net 97)
-	)
-	(segment
-		(start 149.225 120.25)
-		(end 149.225 106.9975)
-		(width 0.2)
-		(layer "B.Cu")
-		(net 97)
-	)
-	(segment
 		(start 139.7 106.3625)
 		(end 140.49375 107.15625)
@@
 	)
 	(segment
-		(start 209.901835 124.6475)
-		(end 206.298085 121.04375)
+		(start 254.98125 124.6475)
+		(end 209.901835 124.6475)
 		(width 0.2)
 		(layer "B.Cu")
@@
 		(width 0.2)
 		(layer "B.Cu")
+		(net 97)
+	)
+	(segment
+		(start 203.621835 118.3675)
+		(end 149.3925 118.3675)
+		(width 0.2)
+		(layer "B.Cu")

Commit message: more footprint stuff
Parts:
- SW1, SW10, SW11, SW13, SW14, SW15, SW16, SW17, SW19, SW2, SW20, SW21, SW22, SW23, SW25, SW26, SW27, SW28, SW29, SW31, SW32, SW33, SW34, SW35, SW37, SW38, SW39, SW40, SW41, SW43, SW44, SW45, SW46, SW47, SW49, SW50, SW51, SW52, SW53, SW54, SW55, SW56, SW57, SW58, SW59, SW60, SW61, SW62, SW63, SW64, SW65, SW66, SW67, SW68, SW69, SW7, SW70, SW72, SW73, SW74, SW75, SW77, SW78, SW79, SW8, SW82, SW83, SW84, SW85, SW86, SW87, SW88, SW89, SW9: footprint Button_Switch_Keyboard:SW_Cherry_MX_1.00u_PCB -> Library:SW_Cherry_MX_1.00u_PCB
- SW12, SW18, SW24, SW36, SW42, SW48, SW6: footprint Button_Switch_Keyboard:SW_Cherry_MX_1.25u_PCB -> Library:SW_Cherry_MX_1.25u_PCB
- SW3, SW81: footprint Button_Switch_Keyboard:SW_Cherry_MX_1.50u_PCB -> Library:SW_Cherry_MX_1.50u_PCB
- SW30: footprint Button_Switch_Keyboard:SW_Cherry_MX_6.25u_PCB -> Library:SW_Cherry_MX_6.25u_PCB
- SW4: footprint Button_Switch_Keyboard:SW_Cherry_MX_1.75u_PCB -> Library:SW_Cherry_MX_1.75u_PCB
- SW5, SW76: footprint Button_Switch_Keyboard:SW_Cherry_MX_2.25u_PCB -> Library:SW_Cherry_MX_2.25u_PCB
- SW71: footprint Button_Switch_Keyboard:SW_Cherry_MX_2.75u_PCB -> Library:SW_Cherry_MX_2.75u_PCB
- SW80: footprint Button_Switch_Keyboard:SW_Cherry_MX_2.00u_PCB -> Library:SW_Cherry_MX_2.00u_PCB
